Commit message: spawn my_rb1 robot inside simulation

File: my_rb1_description/urdf/my_rb1_robot.urdf (robot description, URDF)
Before this commit: robot my_rb1, 7 links, 6 joints
Links:
- link left_wheel: mass None -> 1e-3
- link right_wheel: mass None -> 1e-3

Commit message: add differtial drive conroller and laser scaner plugina

File: my_rb1_description/urdf/my_rb1_robot.urdf (robot description, URDF)
Before this commit: robot my_rb1, 7 links, 6 joints
Links:
- link right_wheel: mass 1e-3 -> 1

Commit message: fix issues in robot URDF model

File: my_rb1_description/urdf/my_rb1_robot.urdf (robot description, URDF)
Before this commit: robot my_rb1, 7 links, 6 joints
Links:
- link left_wheel: mass 1e-3 -> 1; geometry collision cylinder length=0.02 radius=0.025; visual cylinder length=0.02 radius=0.025
